Commit message: joint limits

File: 3DOF-WORM/3DOF-WORM.urdf (robot description, URDF)
Before this commit: robot 3DOF_WORM, 4 links, 3 joints
Links:
- removed link link1
- removed link link2
- removed link link3
- removed link link4
- added link link-1; visual mesh filename=./link-1.gltf
- added link link-2; visual mesh filename=./link-2.gltf
- added link link-3; visual mesh filename=./link-3.gltf
- added link link-4; visual mesh filename=./link-4.gltf
Joints:
- removed joint joint1
- removed joint joint2
- removed joint joint3
- added joint joint-1: type revolute, parent link-1, child link-2, origin xyz=0 0 0.1004 rpy=0 0 0, axis 1 0 0, limit lower=-1.57 upper=1.57 effort=120 velocity=5.02654824
- added joint joint-2: type revolute, parent link-2, child link-3, origin xyz=0 0 0.255 rpy=0 0 0, axis 0 1 0, limit lower=-2.094 upper=2.094 effort=120 velocity=5.02654824
- added joint joint-3: type revolute, parent link-3, child link-4, origin xyz=0 0 0.22 rpy=0 0 0, axis 0 1 0, limit lower=-2.094 upper=2.094 effort=120 velocity=5.02654824
