Commit message: Last push from Deepnote

File: URDFs/Pallet-3DOF.urdf (robot description, URDF)
Before this commit: robot Pallet-3DOF, 5 links, 4 joints
Links:
- link link-1: geometry visual mesh filename=../Meshes/link-1.obj
- link link-2: geometry visual mesh filename=../Meshes/link-2.obj
- link link-3: geometry visual mesh filename=../Meshes/link-3.obj
- link link-4: geometry visual mesh filename=../Meshes/link-4.obj

File: URDFs/robot.urdf (robot description, URDF)
Before this commit: robot rrr_description, 5 links, 4 joints
Links:
- added link moon_terrain; visual mesh filename=../Meshes/3d-model.obj
- link link-1: geometry visual mesh filename=../Meshes/link-1.obj
- link link-2: geometry visual mesh filename=../Meshes/link-2.obj
- link link-3: geometry visual mesh filename=../Meshes/link-3.obj
- link link-4: geometry visual mesh filename=../Meshes/link-4.obj
Joints:
- added joint moon_terrain_joint: type fixed, parent world, child moon_terrain, origin xyz=0 0 0 rpy=0 0 0
