Commit message: Fixed mesh paths

File: URDFs/3DOF-WORM.urdf (robot description, URDF)
Before this commit: robot 3DOF-WORM, 4 links, 3 joints
Links:
- link link-1: geometry visual mesh filename=../Meshes/link-1.gltf
- link link-2: geometry visual mesh filename=../Meshes/link-2.gltf
- link link-3: geometry visual mesh filename=../Meshes/link-3.gltf
- link link-4: geometry visual mesh filename=../Meshes/link-4.gltf

Commit message: Simulation dynamics, collision, and inertia

File: URDFs/3DOF-WORM.urdf (robot description, URDF)
Before this commit: robot 3DOF-WORM, 4 links, 3 joints
Links:
- link link-1: mass None -> 3.5; geometry collision cylinder length=0.075 radius=0.06; collision cylinder length=0.11 radius=0.075
- link link-2: mass None -> 3.5; geometry collision box size=0.1 0.08 0.22; collision cylinder length=0.075 radius=0.06
- link link-3: mass None -> 3.5; geometry collision box size=0.08 0.1 0.18; collision cylinder length=0.075 radius=0.06
- link link-4: mass None -> 11; geometry collision box size=0.11 0.15 0.45; collision cylinder length=0.08 radius=0.075
Joints:
- joint joint-1: origin xyz=0 0 0.1004 rpy=0 0 0 -> xyz=0 0 0.145 rpy=0 0 0

Commit message: Fixed lbs vs N conversion issue

File: URDFs/3DOF-WORM.urdf (robot description, URDF)
Before this commit: robot 3DOF-WORM, 4 links, 3 joints
Links:
- link link-1: mass 3.5 -> 1.59
- link link-2: mass 3.5 -> 1.59
- link link-3: mass 3.5 -> 1.59
- link link-4: mass 11 -> 5.00

Commit message: Updated WORM gltfs

File: URDFs/3DOF-WORM.urdf (robot description, URDF)
Before this commit: robot 3DOF-WORM, 4 links, 3 joints
Links:
- link link-1: geometry collision cylinder length=0.075 radius=0.06; collision cylinder length=0.11 radius=0.075
- link link-2: geometry collision box size=0.1 0.08 0.22; collision cylinder length=0.075 radius=0.06
- link link-3: geometry collision box size=0.08 0.1 0.18; collision cylinder length=0.075 radius=0.06
- link link-4: geometry collision box size=0.11 0.15 0.45; collision cylinder length=0.08 radius=0.075
