Commit message: full pallet with 6 worms

File: URDFs/robot.urdf (robot description, URDF)
Before this commit: robot rrr_description, 6 links, 5 joints
Links:
- removed link link-1
- removed link link-2
- removed link link-3
- removed link link-4
- added link foot-1, mass 1.06; collision cylinder length=0.07 radius=0.125; visual mesh filename=../Meshes/foot.gltf
- added link foot-2, mass 1.06; collision cylinder length=0.07 radius=0.125; visual mesh filename=../Meshes/foot.gltf
- added link foot-3, mass 1.06; collision cylinder length=0.07 radius=0.125; visual mesh filename=../Meshes/foot.gltf
- added link foot-4, mass 1.06; collision cylinder length=0.07 radius=0.125; visual mesh filename=../Meshes/foot.gltf
- added link foot-5, mass 1.06; collision cylinder length=0.07 radius=0.125; visual mesh filename=../Meshes/foot.gltf
- added link foot-6, mass 1.06; collision cylinder length=0.07 radius=0.125; visual mesh filename=../Meshes/foot.gltf
- added link link-1.1, mass 1.59; collision cylinder length=0.075 radius=0.06; collision cylinder length=0.11 radius=0.075
- added link link-1.2, mass 1.59; collision box size=0.1 0.08 0.22; collision cylinder length=0.075 radius=0.06
- added link link-1.3, mass 1.59; collision box size=0.08 0.1 0.18; collision cylinder length=0.075 radius=0.06
- added link link-1.4, mass 5.0; collision box size=0.11 0.15 0.45; collision cylinder length=0.08 radius=0.075
- added link link-2.1, mass 1.59; collision cylinder length=0.075 radius=0.06; collision cylinder length=0.11 radius=0.075
- added link link-2.2, mass 1.59; collision box size=0.1 0.08 0.22; collision cylinder length=0.075 radius=0.06
- added link link-2.3, mass 1.59; collision box size=0.08 0.1 0.18; collision cylinder length=0.075 radius=0.06
- added link link-2.4, mass 5.0; collision box size=0.11 0.15 0.45; collision cylinder length=0.08 radius=0.075
- added link link-3.1, mass 1.59; collision cylinder length=0.075 radius=0.06; collision cylinder length=0.11 radius=0.075
- added link link-3.2, mass 1.59; collision box size=0.1 0.08 0.22; collision cylinder length=0.075 radius=0.06
- added link link-3.3, mass 1.59; collision box size=0.08 0.1 0.18; collision cylinder length=0.075 radius=0.06
- added link link-3.4, mass 5.0; collision box size=0.11 0.15 0.45; collision cylinder length=0.08 radius=0.075
- added link link-4.1, mass 1.59; collision cylinder length=0.075 radius=0.06; collision cylinder length=0.11 radius=0.075
- added link link-4.2, mass 1.59; collision box size=0.1 0.08 0.22; collision cylinder length=0.075 radius=0.06
- added link link-4.3, mass 1.59; collision box size=0.08 0.1 0.18; collision cylinder length=0.075 radius=0.06
- added link link-4.4, mass 5.0; collision box size=0.11 0.15 0.45; collision cylinder length=0.08 radius=0.075
- added link link-5.1, mass 1.59; collision cylinder length=0.075 radius=0.06; collision cylinder length=0.11 radius=0.075
- added link link-5.2, mass 1.59; collision box size=0.1 0.08 0.22; collision cylinder length=0.075 radius=0.06
- added link link-5.3, mass 1.59; collision box size=0.08 0.1 0.18; collision cylinder length=0.075 radius=0.06
- added link link-5.4, mass 5.0; collision box size=0.11 0.15 0.45; collision cylinder length=0.08 radius=0.075
- added link link-6.1, mass 1.59; collision cylinder length=0.075 radius=0.06; collision cylinder length=0.11 radius=0.075
- added link link-6.2, mass 1.59; collision box size=0.1 0.08 0.22; collision cylinder length=0.075 radius=0.06
- added link link-6.3, mass 1.59; collision box size=0.08 0.1 0.18; collision cylinder length=0.075 radius=0.06
- added link link-6.4, mass 5.0; collision box size=0.11 0.15 0.45; collision cylinder length=0.08 radius=0.075
- link pallet: geometry collision box size=0.40 0.55 0.455; collision box size=0.45 0.80 0.25
Joints:
- removed joint link1_joint
- removed joint link2_joint
- removed joint link3_joint
- removed joint moon_terrain_joint
- removed joint pallet_joint
- added joint foot-joint1: type fixed, parent link-1.4, child foot-1, origin xyz=0 0.025 0.50 rpy=0 3.14 0
- added joint foot-joint2: type fixed, parent link-2.4, child foot-2, origin xyz=0 0.025 0.50 rpy=0 3.14 0
- added joint foot-joint3: type fixed, parent link-3.4, child foot-3, origin xyz=0 0.025 0.50 rpy=0 3.14 0
- added joint foot-joint4: type fixed, parent link-4.4, child foot-4, origin xyz=0 0.025 0.50 rpy=0 3.14 0
- added joint foot-joint5: type fixed, parent link-5.4, child foot-5, origin xyz=0 0.025 0.50 rpy=0 3.14 0
- added joint foot-joint6: type fixed, parent link-6.4, child foot-6, origin xyz=0 0.025 0.50 rpy=0 3.14 0
- added joint joint-1.1: type revolute, parent link-1.1, child link-1.2, origin xyz=0 0 0.145 rpy=0 0 0, axis 1 0 0, limit lower=-1.57 upper=1.57 effort=120 velocity=5.02654824
- added joint joint-1.2: type revolute, parent link-1.2, child link-1.3, origin xyz=0 0 0.255 rpy=0 0 0, axis 0 1 0, limit lower=-2.094 upper=2.094 effort=120 velocity=5.02654824
- added joint joint-1.3: type revolute, parent link-1.3, child link-1.4, origin xyz=0 0 0.22 rpy=0 0 0, axis 0 1 0, limit lower=-2.094 upper=2.094 effort=120 velocity=5.02654824
- added joint joint-2.1: type revolute, parent link-2.1, child link-2.2, origin xyz=0 0 0.145 rpy=0 0 0, axis 1 0 0, limit lower=-1.57 upper=1.57 effort=120 velocity=5.02654824
- added joint joint-2.2: type revolute, parent link-2.2, child link-2.3, origin xyz=0 0 0.255 rpy=0 0 0, axis 0 1 0, limit lower=-2.094 upper=2.094 effort=120 velocity=5.02654824
- added joint joint-2.3: type revolute, parent link-2.3, child link-2.4, origin xyz=0 0 0.22 rpy=0 0 0, axis 0 1 0, limit lower=-2.094 upper=2.094 effort=120 velocity=5.02654824
- added joint joint-3.1: type revolute, parent link-3.1, child link-3.2, origin xyz=0 0 0.145 rpy=0 0 0, axis 1 0 0, limit lower=-1.57 upper=1.57 effort=120 velocity=5.02654824
- added joint joint-3.2: type revolute, parent link-3.2, child link-3.3, origin xyz=0 0 0.255 rpy=0 0 0, axis 0 1 0, limit lower=-2.094 upper=2.094 effort=120 velocity=5.02654824
- added joint joint-3.3: type revolute, parent link-3.3, child link-3.4, origin xyz=0 0 0.22 rpy=0 0 0, axis 0 1 0, limit lower=-2.094 upper=2.094 effort=120 velocity=5.02654824
- added joint joint-4.1: type revolute, parent link-4.1, child link-4.2, origin xyz=0 0 0.145 rpy=0 0 0, axis 1 0 0, limit lower=-1.57 upper=1.57 effort=120 velocity=5.02654824
- added joint joint-4.2: type revolute, parent link-4.2, child link-4.3, origin xyz=0 0 0.255 rpy=0 0 0, axis 0 1 0, limit lower=-2.094 upper=2.094 effort=120 velocity=5.02654824
- added joint joint-4.3: type revolute, parent link-4.3, child link-4.4, origin xyz=0 0 0.22 rpy=0 0 0, axis 0 1 0, limit lower=-2.094 upper=2.094 effort=120 velocity=5.02654824
- added joint joint-5.1: type revolute, parent link-5.1, child link-5.2, origin xyz=0 0 0.145 rpy=0 0 0, axis 1 0 0, limit lower=-1.57 upper=1.57 effort=120 velocity=5.02654824
- added joint joint-5.2: type revolute, parent link-5.2, child link-5.3, origin xyz=0 0 0.255 rpy=0 0 0, axis 0 1 0, limit lower=-2.094 upper=2.094 effort=120 velocity=5.02654824
- added joint joint-5.3: type revolute, parent link-5.3, child link-5.4, origin xyz=0 0 0.22 rpy=0 0 0, axis 0 1 0, limit lower=-2.094 upper=2.094 effort=120 velocity=5.02654824
- added joint joint-6.1: type revolute, parent link-6.1, child link-6.2, origin xyz=0 0 0.145 rpy=0 0 0, axis 1 0 0, limit lower=-1.57 upper=1.57 effort=120 velocity=5.02654824
- added joint joint-6.2: type revolute, parent link-6.2, child link-6.3, origin xyz=0 0 0.255 rpy=0 0 0, axis 0 1 0, limit lower=-2.094 upper=2.094 effort=120 velocity=5.02654824
- added joint joint-6.3: type revolute, parent link-6.3, child link-6.4, origin xyz=0 0 0.22 rpy=0 0 0, axis 0 1 0, limit lower=-2.094 upper=2.094 effort=120 velocity=5.02654824
- added joint pallet-joint1: type fixed, parent pallet, child link-1.1, origin xyz=0.17 0.33 0.487 rpy=0 1.57 0
- added joint pallet-joint2: type fixed, parent pallet, child link-2.1, origin xyz=0.17 -0.33 0.487 rpy=0 1.57 0
- added joint pallet-joint3: type fixed, parent pallet, child link-3.1, origin xyz=-0.17 -0.33 0.487 rpy=0 -1.57 0
- added joint pallet-joint4: type fixed, parent pallet, child link-4.1, origin xyz=-0.17 0.33 0.487 rpy=0 -1.57 0
- added joint pallet-joint5: type fixed, parent pallet, child link-5.1, origin xyz=0 0.36 0.487 rpy=-1.57 -1.57 0
- added joint pallet-joint6: type fixed, parent pallet, child link-6.1, origin xyz=0 -0.36 0.487 rpy=1.57 1.57 0
- added joint pallet-moon: type fixed, parent moon_terrain, child pallet, origin xyz=0 0 0 rpy=0 0 0

File: XACRO/robot.macro.xacro (robot description, xacro)
@@ -1,9 +1,24 @@
 <?xml version="1.0"?>
-<robot xmlns:xacro="http://www.ros.org/wiki/xacro">
+<robot xmlns:drake="http://drake.mit.edu" xmlns:xacro="http://www.ros.org/wiki/xacro">
 <!-- ================== -->
 <!--     LINK MACROS    -->
 <!-- ================== -->
-<xacro:macro name="link-1" params="name roll">
+<xacro:macro name="moon_terrain">
+    <link name="moon_terrain">
+        <visual>
+            <origin xyz="0 0 0" rpy="0 0 0"/>
+            <geometry>
+                <mesh filename="../Meshes/3d-model.obj"/>
+            </geometry>
+        </visual>
+    </link>
+</xacro:macro>
+<xacro:macro name="link-1" params="name roll inertial_z mass ixx iyy izz base_z base_length base_radius motor_x motor_z motor_pitch motor_length motor_radius ">
     <link name="${name}">
+        <inertial>
+            <origin xyz="0 0 ${inertial_z}" rpy="0 0 0"/>
+            <mass value="${mass}"/>
+            <inertia ixx="${ixx}" ixy="0" ixz="0" iyy="${iyy}" iyz="0" izz="${izz}"/>
+        </inertial>
         <visual>
             <origin xyz="0 0 0" rpy="${roll} 0 0"/>
@@ -12,18 +27,52 @@
             </geometry>
         </visual>
+        <collision name="link-1-base-collision">
+            <origin xyz="0 0 ${base_z}" rpy="0 0 0"/>
+            <geometry>
+                <cylinder length="${base_length}" radius="${base_radius}"/>
+            </geometry>
+        </collision>
+        <collision name="link-1-motor-collision">
+            <origin xyz="${motor_x} 0 ${motor_z}" rpy="0 ${motor_pitch} 0"/>
+            <geometry>
+            <cylinder length="${motor_length}" radius="${motor_radius}"/>
+        </geometry>
+    </collision>
     </link>
 </xacro:macro>
-<xacro:macro name="link-2" params="name pos_x roll">
+<xacro:macro name="link-2" params="name pos_x roll inertial_z mass ixx iyy izz base_x base_z box_x box_y box_z motor_y motor_z motor_roll motor_length motor_radius ">
     <link name="${name}">
+        <inertial>
+            <origin xyz="0 0 ${inertial_z}" rpy="0 0 0"/>
+            <mass value="${mass}"/>
+            <inertia ixx="${ixx}" ixy="0" ixz="0" iyy="${iyy}" iyz="0" izz="${izz}"/>
+        </inertial>
         <visual>
-            <origin xyz="${pos_x} 0.0" rpy="${roll} 0 0"/>
+            <origin xyz="${pos_x} 0 0" rpy="${roll} 0 0"/>
             <geometry>
                 <mesh filename="../Meshes/link-2.gltf"/>
             </geometry>
         </visual>
+        <collision name="link-2-base-collision">
+            <origin xyz="${base_x} 0 ${base_z}" rpy="0 0 0"/>
+            <geometry>
+                <box size="${box_x} ${box_y} ${box_z}"/>
+            </geometry>
+        </collision>
+        <collision name="link-2-motor-collision">
+            <origin xyz="0 ${motor_y} ${motor_z}" rpy="${motor_roll} 0 0"/>
+            <geometry>
+                <cylinder length="${motor_length}" radius="${motor_radius}"/>
+            </geometry>
+        </collision>
     </link>
 </xacro:macro>
-<xacro:macro name="link-3" params="name pos_y roll pitch yaw">
+<xacro:macro name="link-3" params="name pos_y roll pitch mass inertial_z ixx iyy izz base_y base_z box_x box_y box_z motor_y motor_z motor_roll motor_length motor_radius">
     <link name="${name}">
+        <inertial>
+            <origin xyz="0 0 ${inertial_z}" rpy="0 0 0"/>
+            <mass value="${mass}"/>
+            <inertia ixx="${ixx}" ixy="0" ixz="0" iyy="${iyy}" iyz="0" izz="${izz}"/>
+        </inertial>
         <visual>
             <origin xyz="0.0 ${pos_y} 0.0 " rpy="${roll} ${pitch} 0"/>
@@ -32,53 +81,98 @@
             </geometry>
         </visual>
+        <collision name="link-3-base-collision">
+            <origin xyz="0 ${base_y} ${base_z}" rpy="0 0 0"/>
+            <geometry>
+                <box size="${box_x} ${box_y} ${box_z}"/>
+            </geometry>
+        </collision>
+        <collision name="link-3-motor-collision">
+            <origin xyz="0 ${motor_y} ${motor_z}" rpy="${motor_roll} 0 0"/>
+            <geometry>
+                <cylinder length="${motor_length}" radius="${motor_radius}"/>
+            </geometry>
+        </collision>
     </link>
 </xacro:macro>
-<xacro:macro name="link-4" params="name pos_y roll yaw">
-<link name="${name}">
-    <visual>
-        <origin xyz="0 ${pos_y} 0 " rpy="${roll} 0 ${yaw}"/>
-        <geometry>
-            <mesh filename="../Meshes/link-4.gltf"/>
-        </geometry>
-    </visual>
-</link>
+<xacro:macro name="link-4" params="name pos_y roll yaw inertial_y inertial_z mass ixx iyy izz base_y base_z box_x box_y box_z uib_y uib_z uib_length uib_radius">
+    <link name="${name}">
+        <inertial>
+            <origin xyz="0 ${inertial_y} ${inertial_z}" rpy="0 0 0"/>
+            <mass value="${mass}"/>
+            <inertia ixx="${ixx}" ixy="0" ixz="0" iyy="${iyy}" iyz="0" izz="${izz}"/>
+        </inertial>
+        <visual>
+            <origin xyz="0 ${pos_y} 0 " rpy="${roll} 0 ${yaw}"/>
+            <geometry>
+                <mesh filename="../Meshes/link-4.gltf"/>
+            </geometry>
+        </visual>
+        <collision name="link-3-base-collision">
+            <origin xyz="0 ${base_y} ${base_z}" rpy="0 0 0"/>
+            <geometry>
+                <box size="${box_x} ${box_y} ${box_z}"/>
+            </geometry>
+        </collision>
+        <collision name="link-1-uib-collision">
+            <origin xyz="0 ${uib_y} ${uib_z}" rpy="0 0 0"/>
+            <geometry>
+                <cylinder length="${uib_length}" radius="${uib_radius}"/>
+            </geometry>
+        </collision>
+    </link>
 </xacro:macro>
 <xacro:macro name="pallet" params="name pos_z roll">
-<link name="${name}">
-    <visual>
-        <origin xyz="0 0 ${pos_z}" rpy="${roll} 0 0"/>
-        <geometry>
-            <mesh filename="../Meshes/pallet.gltf"/>
-        </geometry>
-    </visual>
-</link>
+    <link name="${name}">
+        <visual>
+            <origin xyz="0 0 ${pos_z}" rpy="${roll} 0 0"/>
+            <geometry>
+                <mesh filename="../Meshes/pallet.gltf"/>
+            </geometry>
+        </visual>
+    </link>
 </xacro:macro>
 <!-- ================== -->
 <!--     JOINT MACROS   -->
 <!-- ================== -->
-<xacro:macro name="fixed_joint" params="name parent child pos_x pos_y pos_z">
-<joint name="${name}" type="fixed">
-    <parent link="${parent}"/>
-    <child link="${child}"/>
-    <origin rpy="0 1.57 0" xyz="${pos_x} ${pos_y} ${pos_z}"/>
+<xacro:macro name="fixed_joint" params="name parent child pos_x pos_y pos_z roll pitch">
+    <joint name="${name}" type="fixed">
+        <parent link="${parent}"/>
+        <child link="${child}"/>
+        <origin rpy="${roll} ${pitch} 0" xyz="${pos_x} ${pos_y} ${pos_z}"/>
+        </joint>
+</xacro:macro>
+<xacro:macro name="revolute_joint" params="name parent child axis pos_z lower upper effort velocity">
+    <joint name="${name}" type="revolute">
+        <parent link="${parent}"/>
+        <child link="${child}"/>
+        <xacro:if value="${axis == 'x'}">
+            <axis xyz="1 0 0"/>
+        </xacro:if>
+        <xacro:if value="${axis == 'y'}">
+            <axis xyz="0 1 0"/>
+        </xacro:if>
+        <xacro:if value="${axis == 'z'}">
+            <axis xyz="0 0 1"/>
+        </xacro:if>
+        <origin rpy="0 0 0" xyz="0 0 ${pos_z}"/>
+        <limit effort="${effort}" lower="${lower}" upper="${upper}" velocity="${velocity}"/>
+        <dynamics damping="0.8487"/>
     </joint>
 </xacro:macro>
-<xacro:macro name="revolute_joint" params="name parent child axis pos_z lower upper effort velocity">
-<joint name="${name}" type="revolute">
-    <parent link="${parent}"/>
-    <child link="${child}"/>
-    <xacro:if value="${axis == 'x'}">
-        <axis xyz="1 0 0"/>
-    </xacro:if>
-    <xacro:if value="${axis == 'y'}">
-        <axis xyz="0 1 0"/>
-    </xacro:if>
-    <xacro:if value="${axis == 'z'}">
-        <axis xyz="0 0 1"/>
-    </xacro:if>
-    <origin rpy="0 0 0" xyz="0 0 ${pos_z}"/>
-    <limit effort="${effort}" lower="${lower}" upper="${upper}" velocity="${velocity}"/>
-    <dynamics damping="1"/>
-</joint>
+<!-- Define a macro for transmissions -->
+<xacro:macro name="create_transmission" params="transmission_name joint_name actuator_name">
+    <transmission name="${transmission_name}">
+        <robotNamespace>/3DOF-WORM</robotNamespace>
+        <type>transmission_interface/SimpleTransmission</type>
+        <joint name="${joint_name}">
+            <hardwareInterface>PositionJointInterface</hardwareInterface>
+        </joint>
+        <actuator name="${actuator_name}">
+            <hardwareInterface>PositionJointInterface</hardwareInterface>
+            <mechanicalReduction>1</mechanicalReduction>
+            <drake:gear_ratio value="64.0" />
+            <drake:rotor_inertia value="0.00005645" />
+        </actuator>
+    </transmission>
 </xacro:macro>
 </robot>
