Commit message: Updated pallet mesh, updated pallet collision, added offset option, populated correct mass/inertia fields. Still need to include shoes on model.

File: URDFs/turtle.urdf (robot description, URDF)
Before this commit: robot turtle, 27 links, 27 joints
Links:
- added link virtual_turtle_body
- link turtle_body: mass 1.59 -> 21.89; geometry collision box size=0.11 0.11 0.4; collision box size=0.8 0.4 0.02
Joints:
- removed joint temp
- added joint virtual_turtle_body_joint_fixed: type fixed, parent virtual_turtle_body, child turtle_body, origin xyz=0 0 1.35

File: XACRO/pallets.macro.xacro (robot description, xacro)
@@ -8,15 +8,18 @@
 <!-- |      back_left_uib,  back_right_uib,  back_center_uib                           | -->
 <!-- =================================================================================== -->
-<xacro:macro name="turtle">
-    <joint name="temp" type="fixed">
-        <parent link="world"/>
+<xacro:macro name="turtle" params="spawn_z">
+    <!-- Virtual link to offset the body by some fixed amount -->
+    <link name="virtual_turtle_body"/>
+    <joint name="virtual_turtle_body_joint_fixed" type="fixed">
+        <parent link="virtual_turtle_body"/>
         <child link="turtle_body"/>
+        <origin xyz="0 0 ${spawn_z}"/>
     </joint>
     <!-- Main pallet -->
     <link name="turtle_body">
         <inertial>
-            <origin xyz="0 0 0.0725" rpy="0 0 0"/>
-            <mass value="1.59"/>
-            <inertia ixx="0.010" ixy="0" ixz="0" iyy="0.010" iyz="0" izz="0.011"/>
+            <origin xyz="0 0 -0.13" rpy="0 0 -1.57"/>
+            <mass value="21.89"/>
+            <inertia ixx="0.9" ixy="0" ixz="0" iyy="1.5" iyz="0" izz="1.0"/>
         </inertial>
         <visual>
@@ -30,4 +33,16 @@
             <geometry>
                 <box size="0.8 0.4 0.15"/>
+            </geometry>
+        </collision>
+        <collision name="turtle_stand_collision">
+            <origin xyz="0 0 -0.2" rpy="0 0 0"/>
+            <geometry>
+                <box size="0.11 0.11 0.4"/>
+            </geometry>
+        </collision>
+        <collision name="turtle_plate_collision">
+            <origin xyz="0 0 -0.4" rpy="0 0 0"/>
+            <geometry>
+                <box size="0.8 0.4 0.02"/>
             </geometry>
         </collision>

File: XACRO/turtle.urdf.xacro (robot description, xacro)
@@ -10,5 +10,5 @@
 <xacro:include filename="pallets.macro.xacro"/>
 <!-- Create a turtle pallet and attach worms to each corner uib -->
-<xacro:turtle/>
+<xacro:turtle spawn_z="1.35"/>
 <xacro:worm namespace="$(eval front_left)" parent_link="front_left_uib" base_xyz="0 0 0" base_rpy="0 0 0"/>
 <xacro:worm namespace="$(eval front_right)" parent_link="front_right_uib" base_xyz="0 0 0" base_rpy="0 0 0"/>
