Commit message: Fixed xacro to prevent floating links when connected to world, recompiled pony-worm urdf with updated params

File: URDFs/pony-worm.urdf (robot description, URDF)
Before this commit: robot worm, 5 links, 4 joints
Joints:
- removed joint pony_joint_fixed_0
- added joint pony_base_joint_fixed: type fixed, parent pony_base, child pony_link_0
- added joint pony_uib_joint_fixed: type fixed, parent world, child pony_base, origin xyz=0 0 0 rpy=0 0 0

File: XACRO/3dof-worm.macro.xacro (robot description, xacro)
@@ -1,6 +1,14 @@
 <?xml version="1.0"?>
 <robot xmlns:drake="http://drake.mit.edu" xmlns:xacro="http://www.ros.org/wiki/xacro">
-<!-- Macro for an entire worm -->
-<xacro:macro name="worm" params="namespace base_link base_xyz base_rpy">
+<!--
+//  Macro for an entire worm model with simple geometry collision.
+//
+//  Args:
+//      namespace: namespace that this worm publishes to
+//      parent_link: link name to affix the uib of this worm to
+//      base_xyz: translational offset of uib, ex: "0.2 0.1 0.1"
+//      base_rpy: rotational offset of uib, "0.2 0.1 0.1"
+-->
+<xacro:macro name="worm" params="namespace parent_link base_xyz base_rpy">
     <!-- Local parameters -->
     <xacro:property name="motor_collision_length" value="0.075"/>
@@ -11,9 +19,13 @@
     <xacro:property name="motor_gear_ratio" value="64"/>
     <xacro:property name="motor_rotor_inertia" value="0.00005645"/>
+    <joint name="${namespace}_uib_joint_fixed" type="fixed">
+        <parent link="${parent_link}"/>
+        <child link="${namespace}_base"/>
+        <origin xyz="${base_xyz}" rpy="${base_rpy}"/>
+    </joint>
     <link name="${namespace}_base"/>
-    <joint name="${namespace}_joint_fixed_0" type="fixed">
-        <parent link="${base_link}"/>
+    <joint name="${namespace}_base_joint_fixed" type="fixed">
+        <parent link="${namespace}_base"/>
         <child link="${namespace}_link_0"/>
-        <origin xyz="${base_xyz}" rpy="${base_rpy}"/>
     </joint>
     <link name="${namespace}_link_0">

File: XACRO/3dof-worm.urdf.xacro (robot description, xacro)
@@ -9,4 +9,4 @@
 <xacro:include filename="3dof-worm.macro.xacro"/>
 <!-- Create a default worm fixed at the origin with the name passed -->
-<xacro:worm namespace="$(eval name)" base_link="world" base_xyz="0 0 0" base_rpy="0 0 0"/>
+<xacro:worm namespace="$(eval name)" parent_link="world" base_xyz="0 0 0" base_rpy="0 0 0"/>
 </robot>

Commit message: Change worm joint limit

File: URDFs/pony-worm.urdf (robot description, URDF)
Before this commit: robot worm, 5 links, 5 joints
Joints:
- joint pony_joint_0: limit lower=-1.57 upper=1.57 effort=120 velocity=5.02654824 -> lower=-2.094 upper=2.094 effort=120 velocity=5.02654824

File: XACRO/3dof-worm.macro.xacro (robot description, xacro)
@@ -1,13 +1,12 @@
 <?xml version="1.0"?>
 <robot xmlns:drake="http://drake.mit.edu" xmlns:xacro="http://www.ros.org/wiki/xacro">
-<!--
-//  Macro for an entire worm model with simple geometry collision.
-//
-//  Args:
-//      namespace: namespace that this worm publishes to
-//      parent_link: link name to affix the uib of this worm to
-//      base_xyz: translational offset of uib, ex: "0.2 0.1 0.1"
-//      base_rpy: rotational offset of uib, "0.2 0.1 0.1"
--->
+<!-- =================================================================================== -->
+<!-- |    Macro for an entire worm model with simple geometry collision.               | -->
+<!-- |    Args:                                                                        | -->
+<!-- |      namespace: namespace that this worm publishes to                           | -->
+<!-- |      parent_link: link name to affix the uib of this worm to                    | -->
+<!-- |      base_xyz: translational offset of uib, ex: "0.2 0.1 0.1"                   | -->
+<!-- |      base_rpy: rotational offset of uib, "0.2 0.1 0.1"                          | -->
+<!-- =================================================================================== -->
 <xacro:macro name="worm" params="namespace parent_link base_xyz base_rpy">
     <!-- Local parameters -->
@@ -59,5 +58,5 @@
         <origin xyz="0 0 0.145" rpy="0 0 0" />
         <axis xyz="1 0 0" />
-        <limit lower="-1.57" upper="1.57" effort="${motor_effort_limit}" velocity="${motor_velocity_limit}"/>
+        <limit lower="-2.094" upper="2.094" effort="${motor_effort_limit}" velocity="${motor_velocity_limit}"/>
         <dynamics damping="${motor_damping}"/>
     </joint>

Commit message: Fixed mirroring issue in 3dof models. Fixed bug in turtle urdf macroof sides being swapped

File: URDFs/pony-worm.urdf (robot description, URDF)
Before this commit: robot worm, 5 links, 5 joints
Joints:
- joint pony_joint_1: origin xyz=0 0 0.255 rpy=0 0 0 -> xyz=0 0 0.25 rpy=0 0 0

File: URDFs/turtle.urdf (robot description, URDF)
Before this commit: robot turtle, 27 links, 27 joints
Joints:
- joint back_left_uib_joint_fixed: origin xyz=-0.328 -0.204 0.062 rpy=1.57 -1.57 0 -> xyz=-0.328 0.204 0.062 rpy=-1.57 1.57 0
- joint back_right_uib_joint_fixed: origin xyz=-0.328 0.204 0.062 rpy=-1.57 -1.57 0 -> xyz=-0.328 -0.204 0.062 rpy=1.57 -1.57 0
- joint duck_joint_1: origin xyz=0 0 0.255 rpy=0 0 0 -> xyz=0 0 0.25 rpy=0 0 0
- joint frog_joint_1: origin xyz=0 0 0.255 rpy=0 0 0 -> xyz=0 0 0.25 rpy=0 0 0
- joint front_left_uib_joint_fixed: origin xyz=0.328 -0.204 0.062 rpy=1.57 -1.57 0 -> xyz=0.328 0.204 0.062 rpy=-1.57 1.57 0
- joint front_right_uib_joint_fixed: origin xyz=0.328 0.204 0.062 rpy=-1.57 -1.57 0 -> xyz=0.328 -0.204 0.062 rpy=1.57 -1.57 0
- joint lion_joint_1: origin xyz=0 0 0.255 rpy=0 0 0 -> xyz=0 0 0.25 rpy=0 0 0
- joint pony_joint_1: origin xyz=0 0 0.255 rpy=0 0 0 -> xyz=0 0 0.25 rpy=0 0 0

File: XACRO/3dof-worm.macro.xacro (robot description, xacro)
@@ -80,5 +80,5 @@
         </collision>
         <collision name="${namespace}_link_1_motor_collision">
-            <origin xyz="0 0.008 0.255" rpy="1.57 0 0"/>
+            <origin xyz="0 -0.008 0.255" rpy="1.57 0 0"/>
             <geometry>
                 <cylinder length="${motor_collision_length}" radius="${motor_collision_radius}"/>
@@ -89,5 +89,5 @@
         <parent link="${namespace}_link_1"/>
         <child link="${namespace}_link_2"/>
-        <origin xyz="0 0 0.255" rpy="0 0 0" />
+        <origin xyz="0 0 0.25" rpy="0 0 0" />
         <axis xyz="0 1 0" />
         <limit lower="-2.094" upper="2.094" effort="${motor_effort_limit}" velocity="${motor_velocity_limit}"/>
@@ -101,5 +101,5 @@
         </inertial>
         <visual>
-            <origin xyz="0 0.05 0" rpy="0 0 0"/>
+            <origin xyz="0 -0.05 0" rpy="0 0 3.14"/>
             <geometry>
                 <mesh filename="../Meshes/link-2.gltf"/>
@@ -107,5 +107,5 @@
         </visual>
         <collision name="${namespace}_link_2_base_collision">
-            <origin xyz="0 0.01 0.07" rpy="0 0 0"/>
+            <origin xyz="0 -0.01 0.07" rpy="0 0 0"/>
             <geometry>
                 <box size="0.08 0.1 0.18"/>

File: XACRO/pallets.macro.xacro (robot description, xacro)
@@ -34,16 +34,16 @@
     </link>
     <!-- Front UIBs -->
+    <joint name="front_left_uib_joint_fixed" type="fixed">
+        <parent link="turtle_body"/>
+        <child link="front_left_uib"/>
+        <origin xyz="0.328 0.204 0.062" rpy="-1.57 1.57 0"/>
+    </joint>
+    <link name="front_left_uib"/>
     <joint name="front_right_uib_joint_fixed" type="fixed">
         <parent link="turtle_body"/>
         <child link="front_right_uib"/>
-        <origin xyz="0.328 0.204 0.062" rpy="-1.57 -1.57 0"/>
+        <origin xyz="0.328 -0.204 0.062" rpy="1.57 -1.57 0"/>
     </joint>
     <link name="front_right_uib"/>
-    <joint name="front_left_uib_joint_fixed" type="fixed">
-        <parent link="turtle_body"/>
-        <child link="front_left_uib"/>
-        <origin xyz="0.328 -0.204 0.062" rpy="1.57 -1.57 0"/>
-    </joint>
-    <link name="front_left_uib"/>
     <joint name="front_center_uib_joint_fixed" type="fixed">
         <parent link="turtle_body"/>
@@ -53,16 +53,16 @@
     <link name="front_center_uib"/>
     <!-- Back UIBs -->
+    <joint name="back_left_uib_joint_fixed" type="fixed">
+        <parent link="turtle_body"/>
+        <child link="back_left_uib"/>
+        <origin xyz="-0.328 0.204 0.062" rpy="-1.57 1.57 0"/>
+    </joint>
+    <link name="back_left_uib"/>
     <joint name="back_right_uib_joint_fixed" type="fixed">
         <parent link="turtle_body"/>
         <child link="back_right_uib"/>
-        <origin xyz="-0.328 0.204 0.062" rpy="-1.57 -1.57 0"/>
+        <origin xyz="-0.328 -0.204 0.062" rpy="1.57 -1.57 0"/>
     </joint>
     <link name="back_right_uib"/>
-    <joint name="back_left_uib_joint_fixed" type="fixed">
-        <parent link="turtle_body"/>
-        <child link="back_left_uib"/>
-        <origin xyz="-0.328 -0.204 0.062" rpy="1.57 -1.57 0"/>
-    </joint>
-    <link name="back_left_uib"/>
     <joint name="back_center_uib_joint_fixed" type="fixed">
         <parent link="turtle_body"/>

Commit message: Added foot module with collision. parent_link -> downstream links organization

File: URDFs/pony-worm.urdf (robot description, URDF)
Before this commit: robot worm, 5 links, 5 joints
Links:
- added link pony_end_uib
Joints:
- added joint pony_end_uib_joint_fixed: type fixed, parent pony_link_3, child pony_end_uib, origin xyz=0 -0.012 0.498 rpy=3.14 0 -0.35

File: URDFs/turtle.urdf (robot description, URDF)
Before this commit: robot turtle, 28 links, 27 joints
Links:
- added link duck_end_uib
- added link duck_rubber_foot, mass 1.54; collision cylinder length=0.018 radius=0.115; collision cylinder length=0.05 radius=0.07
- added link frog_end_uib
- added link frog_rubber_foot, mass 1.54; collision cylinder length=0.018 radius=0.115; collision cylinder length=0.05 radius=0.07
- added link lion_end_uib
- added link lion_rubber_foot, mass 1.54; collision cylinder length=0.018 radius=0.115; collision cylinder length=0.05 radius=0.07
- added link pony_end_uib
- added link pony_rubber_foot, mass 1.54; collision cylinder length=0.018 radius=0.115; collision cylinder length=0.05 radius=0.07
Joints:
- added joint duck_end_uib_joint_fixed: type fixed, parent duck_link_3, child duck_end_uib, origin xyz=0 -0.012 0.498 rpy=3.14 0 -0.35
- added joint duck_rubber_foot_joint_fixed: type fixed, parent duck_end_uib, child duck_rubber_foot
- added joint frog_end_uib_joint_fixed: type fixed, parent frog_link_3, child frog_end_uib, origin xyz=0 -0.012 0.498 rpy=3.14 0 -0.35
- added joint frog_rubber_foot_joint_fixed: type fixed, parent frog_end_uib, child frog_rubber_foot
- added joint lion_end_uib_joint_fixed: type fixed, parent lion_link_3, child lion_end_uib, origin xyz=0 -0.012 0.498 rpy=3.14 0 -0.35
- added joint lion_rubber_foot_joint_fixed: type fixed, parent lion_end_uib, child lion_rubber_foot
- added joint pony_end_uib_joint_fixed: type fixed, parent pony_link_3, child pony_end_uib, origin xyz=0 -0.012 0.498 rpy=3.14 0 -0.35
- added joint pony_rubber_foot_joint_fixed: type fixed, parent pony_end_uib, child pony_rubber_foot

File: XACRO/3dof-worm.macro.xacro (robot description, xacro)
@@ -3,4 +3,6 @@
 <!-- =================================================================================== -->
 <!-- |    Macro for an entire worm model with simple geometry collision.               | -->
+<!-- |    Downstream Links:                                                            | -->
+<!-- |      {namespace}_end_uib                                                        | -->
 <!-- |    Args:                                                                        | -->
 <!-- |      namespace: namespace that this worm publishes to                           | -->
@@ -152,4 +154,11 @@
         </collision>
     </link>
+    <!-- Downstream link -->
+    <joint name="${namespace}_end_uib_joint_fixed" type="fixed">
+        <parent link="${namespace}_link_3"/>
+        <child link="${namespace}_end_uib"/>
+        <origin xyz="0 -0.012 0.498" rpy="3.14 0 -0.35"/>
+    </joint>
+    <link name="${namespace}_end_uib"/>
     <!-- Transmission definitions -->
     <transmission name="${namespace}_tran_0">

File: XACRO/pallets.macro.xacro (robot description, xacro)
@@ -2,9 +2,14 @@
 <robot xmlns:drake="http://drake.mit.edu" xmlns:xacro="http://www.ros.org/wiki/xacro">
 <!-- =================================================================================== -->
-<!-- |    Macro for a turtle pallet with six uib attachment points. To attach          | -->
-<!-- |    something to a uib, create a joint after calling this macro and set the      | -->
-<!-- |    parent link to one of the following:                                         | -->
-<!-- |      front_left_uib, front_right_uib, front_center_uib                          | -->
-<!-- |      back_left_uib,  back_right_uib,  back_center_uib                           | -->
+<!-- |    Macro for a turtle pallet with six uib attachment points.                    | -->
+<!-- |    Downstream Links:                                                            | -->
+<!-- |      front_left_uib                                                             | -->
+<!-- |      front_right_uib                                                            | -->
+<!-- |      front_center_uib                                                           | -->
+<!-- |      back_left_uib                                                              | -->
+<!-- |      back_right_uib                                                             | -->
+<!-- |      back_center_uib                                                            | -->
+<!-- |    Args:                                                                        | -->
+<!-- |      spawn_z: height (in m) to spawn the pallet at                              | -->
 <!-- =================================================================================== -->
 <xacro:macro name="turtle" params="spawn_z">

File: XACRO/turtle.urdf.xacro (robot description, xacro)
@@ -9,4 +9,5 @@
 <xacro:include filename="3dof-worm.macro.xacro"/>
 <xacro:include filename="pallets.macro.xacro"/>
+<xacro:include filename="species.macro.xacro"/>
 <!-- Create a turtle pallet and attach worms to each corner uib -->
 <xacro:turtle spawn_z="1.35"/>
@@ -15,3 +16,8 @@
 <xacro:worm namespace="$(eval back_left)" parent_link="back_left_uib" base_xyz="0 0 0" base_rpy="0 0 0"/>
 <xacro:worm namespace="$(eval back_right)" parent_link="back_right_uib" base_xyz="0 0 0" base_rpy="0 0 0"/>
+<!-- Attach a foot module to each worm -->
+<xacro:rubber_foot namespace="$(eval front_left)" parent_link="$(eval front_left)_end_uib"/>
+<xacro:rubber_foot namespace="$(eval front_right)" parent_link="$(eval front_right)_end_uib"/>
+<xacro:rubber_foot namespace="$(eval back_left)" parent_link="$(eval back_left)_end_uib"/>
+<xacro:rubber_foot namespace="$(eval back_right)" parent_link="$(eval back_right)_end_uib"/>
 </robot>

Commit message: Add full turtle bot urdf and rubber foot module (#4)
* Basic turtle pallet mesh and xacro. Ideally update model to reflect real robot, body collision not complete, need to add world, temporarily fixing pallet to world for testing.

* Fixed mirroring issue in 3dof models. Fixed bug in turtle urdf macroof sides being swapped

* Rollback motor damping change, model seems highly underdamped compared to real motors

* Updated pallet mesh, updated pallet collision, added offset option, populated correct mass/inertia fields. Still need to include shoes on model.

* Added foot module with collision. parent_link -> downstream links organization

File: URDFs/pony-worm.urdf (robot description, URDF)
Before this commit: robot worm, 5 links, 5 joints
Links:
- added link pony_end_uib
Joints:
- added joint pony_end_uib_joint_fixed: type fixed, parent pony_link_3, child pony_end_uib, origin xyz=0 -0.012 0.498 rpy=3.14 0 -0.35
- joint pony_joint_1: origin xyz=0 0 0.255 rpy=0 0 0 -> xyz=0 0 0.25 rpy=0 0 0

File: XACRO/3dof-worm.macro.xacro (robot description, xacro)
@@ -3,4 +3,6 @@
 <!-- =================================================================================== -->
 <!-- |    Macro for an entire worm model with simple geometry collision.               | -->
+<!-- |    Downstream Links:                                                            | -->
+<!-- |      {namespace}_end_uib                                                        | -->
 <!-- |    Args:                                                                        | -->
 <!-- |      namespace: namespace that this worm publishes to                           | -->
@@ -15,5 +17,5 @@
     <xacro:property name="motor_effort_limit" value="120"/>
     <xacro:property name="motor_velocity_limit" value="5.02654824"/>
-    <xacro:property name="motor_damping" value="0.0028"/>
+    <xacro:property name="motor_damping" value="0.8487"/>
     <xacro:property name="motor_gear_ratio" value="64"/>
     <xacro:property name="motor_rotor_inertia" value="0.00005645"/>
@@ -80,5 +82,5 @@
         </collision>
         <collision name="${namespace}_link_1_motor_collision">
-            <origin xyz="0 0.008 0.255" rpy="1.57 0 0"/>
+            <origin xyz="0 -0.008 0.255" rpy="1.57 0 0"/>
             <geometry>
                 <cylinder length="${motor_collision_length}" radius="${motor_collision_radius}"/>
@@ -89,5 +91,5 @@
         <parent link="${namespace}_link_1"/>
         <child link="${namespace}_link_2"/>
-        <origin xyz="0 0 0.255" rpy="0 0 0" />
+        <origin xyz="0 0 0.25" rpy="0 0 0" />
         <axis xyz="0 1 0" />
         <limit lower="-2.094" upper="2.094" effort="${motor_effort_limit}" velocity="${motor_velocity_limit}"/>
@@ -101,5 +103,5 @@
         </inertial>
         <visual>
-            <origin xyz="0 0.05 0" rpy="0 0 0"/>
+            <origin xyz="0 -0.05 0" rpy="0 0 3.14"/>
             <geometry>
                 <mesh filename="../Meshes/link-2.gltf"/>
@@ -107,5 +109,5 @@
         </visual>
         <collision name="${namespace}_link_2_base_collision">
-            <origin xyz="0 0.01 0.07" rpy="0 0 0"/>
+            <origin xyz="0 -0.01 0.07" rpy="0 0 0"/>
             <geometry>
                 <box size="0.08 0.1 0.18"/>
@@ -152,4 +154,11 @@
         </collision>
     </link>
+    <!-- Downstream link -->
+    <joint name="${namespace}_end_uib_joint_fixed" type="fixed">
+        <parent link="${namespace}_link_3"/>
+        <child link="${namespace}_end_uib"/>
+        <origin xyz="0 -0.012 0.498" rpy="3.14 0 -0.35"/>
+    </joint>
+    <link name="${namespace}_end_uib"/>
     <!-- Transmission definitions -->
     <transmission name="${namespace}_tran_0">
