Commit message: Parameterize mesh type

File: URDFs/pony-worm.urdf (robot description, URDF)
Before this commit: robot worm, 6 links, 6 joints
Links:
- link pony_link_0: geometry collision cylinder length=0.075 radius=0.06; collision cylinder length=0.11 radius=0.075
- link pony_link_1: geometry collision box size=0.1 0.08 0.22; collision cylinder length=0.075 radius=0.06
- link pony_link_2: geometry collision box size=0.08 0.1 0.18; collision cylinder length=0.075 radius=0.06
- link pony_link_3: geometry collision box size=0.11 0.15 0.45; collision cylinder length=0.08 radius=0.075

File: URDFs/turtle.urdf (robot description, URDF)
Before this commit: robot turtle, 36 links, 35 joints
Links:
- link duck_link_0: geometry collision cylinder length=0.075 radius=0.06; collision cylinder length=0.11 radius=0.075
- link duck_link_1: geometry collision box size=0.1 0.08 0.22; collision cylinder length=0.075 radius=0.06
- link duck_link_2: geometry collision box size=0.08 0.1 0.18; collision cylinder length=0.075 radius=0.06
- link duck_link_3: geometry collision box size=0.11 0.15 0.45; collision cylinder length=0.08 radius=0.075
- link duck_rubber_foot: geometry collision cylinder length=0.018 radius=0.115; collision cylinder length=0.05 radius=0.07
- link frog_link_0: geometry collision cylinder length=0.075 radius=0.06; collision cylinder length=0.11 radius=0.075
- link frog_link_1: geometry collision box size=0.1 0.08 0.22; collision cylinder length=0.075 radius=0.06
- link frog_link_2: geometry collision box size=0.08 0.1 0.18; collision cylinder length=0.075 radius=0.06
- link frog_link_3: geometry collision box size=0.11 0.15 0.45; collision cylinder length=0.08 radius=0.075
- link frog_rubber_foot: geometry collision cylinder length=0.018 radius=0.115; collision cylinder length=0.05 radius=0.07
- link lion_link_0: geometry collision cylinder length=0.075 radius=0.06; collision cylinder length=0.11 radius=0.075
- link lion_link_1: geometry collision box size=0.1 0.08 0.22; collision cylinder length=0.075 radius=0.06
- link lion_link_2: geometry collision box size=0.08 0.1 0.18; collision cylinder length=0.075 radius=0.06
- link lion_link_3: geometry collision box size=0.11 0.15 0.45; collision cylinder length=0.08 radius=0.075
- link lion_rubber_foot: geometry collision cylinder length=0.018 radius=0.115; collision cylinder length=0.05 radius=0.07
- link pony_link_0: geometry collision cylinder length=0.075 radius=0.06; collision cylinder length=0.11 radius=0.075
- link pony_link_1: geometry collision box size=0.1 0.08 0.22; collision cylinder length=0.075 radius=0.06
- link pony_link_2: geometry collision box size=0.08 0.1 0.18; collision cylinder length=0.075 radius=0.06
- link pony_link_3: geometry collision box size=0.11 0.15 0.45; collision cylinder length=0.08 radius=0.075
- link pony_rubber_foot: geometry collision cylinder length=0.018 radius=0.115; collision cylinder length=0.05 radius=0.07
- link turtle_body: geometry collision box size=0.11 0.11 0.4; collision box size=0.8 0.4 0.02

File: XACRO/3dof-worm.macro.xacro (robot description, xacro)
@@ -11,5 +11,5 @@
 <!-- |      base_rpy: rotational offset of uib, "0.2 0.1 0.1"                          | -->
 <!-- =================================================================================== -->
-<xacro:macro name="worm" params="namespace parent_link base_xyz base_rpy">
+<xacro:macro name="worm" params="namespace parent_link base_xyz base_rpy mesh_type">
     <!-- Local parameters -->
     <xacro:property name="motor_collision_length" value="0.075"/>
@@ -39,5 +39,5 @@
             <origin xyz="0 0 0.045" rpy="0 0 0"/>
             <geometry>
-                <mesh filename="../Meshes/link-0.gltf"/>
+                <mesh filename="../Meshes/${mesh_type}/link-0.gltf"/>
             </geometry>
         </visual>
@@ -72,5 +72,5 @@
             <origin xyz="0.05 0 0" rpy="0 0 -1.57"/>
             <geometry>
-                <mesh filename="../Meshes/link-1.gltf"/>
+                <mesh filename="../Meshes/${mesh_type}/link-1.gltf"/>
             </geometry>
         </visual>
@@ -105,5 +105,5 @@
             <origin xyz="0 -0.05 0" rpy="0 0 3.14"/>
             <geometry>
-                <mesh filename="../Meshes/link-2.gltf"/>
+                <mesh filename="../Meshes/${mesh_type}/link-2.gltf"/>
             </geometry>
         </visual>
@@ -138,5 +138,5 @@
             <origin xyz="0 -0.05 0" rpy="0 0 1.57"/>
             <geometry>
-                <mesh filename="../Meshes/link-3.gltf"/>
+                <mesh filename="../Meshes/${mesh_type}/link-3.gltf"/>
             </geometry>
         </visual>

File: XACRO/3dof-worm.urdf.xacro (robot description, xacro)
@@ -3,4 +3,5 @@
 <!-- Arguments -->
 <xacro:arg name="name" default=""/>
+<xacro:arg name="mesh_type" default="GLTF"/>
 <xacro:if value="$(eval name == '')">
     <xacro:error msg="'name' was not provided"/>
@@ -9,4 +10,4 @@
 <xacro:include filename="3dof-worm.macro.xacro"/>
 <!-- Create a default worm fixed at the origin with the name passed -->
-<xacro:worm namespace="$(eval name)" parent_link="world" base_xyz="0 0 0" base_rpy="0 0 0"/>
+<xacro:worm namespace="$(eval name)" parent_link="world" base_xyz="0 0 0" base_rpy="0 0 0" mesh_type="$(eval mesh_type)"/>
 </robot>

File: XACRO/pallets.macro.xacro (robot description, xacro)
@@ -13,5 +13,5 @@
 <!-- |      spawn_z: height (in m) to spawn the pallet at                              | -->
 <!-- =================================================================================== -->
-<xacro:macro name="turtle" params="spawn_z">
+<xacro:macro name="turtle" params="spawn_z mesh_type">
     <!-- Virtual link to offset the body by some fixed amount -->
     <link name="virtual_turtle_body"/>
@@ -31,5 +31,5 @@
             <origin xyz="0 0 0" rpy="0 0 -1.57"/>
             <geometry>
-                <mesh filename="../Meshes/turtle-pallet.gltf"/>
+                <mesh filename="../Meshes/${mesh_type}/turtle-pallet.gltf"/>
             </geometry>
         </visual>

File: XACRO/species.macro.xacro (robot description, xacro)
@@ -7,5 +7,5 @@
 <!-- |      parent_link: link name to affix the uib of this module to                  | -->
 <!-- =================================================================================== -->
-<xacro:macro name="rubber_foot" params="namespace parent_link">
+<xacro:macro name="rubber_foot" params="namespace parent_link mesh_type">
     <joint name="${namespace}_rubber_foot_joint_fixed" type="fixed">
         <parent link="${parent_link}"/>
@@ -20,5 +20,5 @@
         <visual>
             <geometry>
-                <mesh filename="../Meshes/rubber-foot.gltf"/>
+                <mesh filename="../Meshes/${mesh_type}/rubber-foot.gltf"/>
             </geometry>
         </visual>

File: XACRO/turtle.urdf.xacro (robot description, xacro)
@@ -6,4 +6,5 @@
 <xacro:arg name="back_left" default="lion"/>
 <xacro:arg name="back_right" default="pony"/>
+<xacro:arg name="mesh_type" default="GLTF"/>
 <!-- Include xacro files -->
 <xacro:include filename="3dof-worm.macro.xacro"/>
@@ -11,13 +12,13 @@
 <xacro:include filename="species.macro.xacro"/>
 <!-- Create a turtle pallet and attach worms to each corner uib -->
-<xacro:turtle spawn_z="1.35"/>
-<xacro:worm namespace="$(eval front_left)" parent_link="front_left_uib" base_xyz="0 0 0" base_rpy="0 0 0"/>
-<xacro:worm namespace="$(eval front_right)" parent_link="front_right_uib" base_xyz="0 0 0" base_rpy="0 0 0"/>
-<xacro:worm namespace="$(eval back_left)" parent_link="back_left_uib" base_xyz="0 0 0" base_rpy="0 0 0"/>
-<xacro:worm namespace="$(eval back_right)" parent_link="back_right_uib" base_xyz="0 0 0" base_rpy="0 0 0"/>
+<xacro:turtle spawn_z="1.35" mesh_type="$(eval mesh_type)"/>
+<xacro:worm namespace="$(eval front_left)" parent_link="front_left_uib" base_xyz="0 0 0" base_rpy="0 0 0" mesh_type="$(eval mesh_type)"/>
+<xacro:worm namespace="$(eval front_right)" parent_link="front_right_uib" base_xyz="0 0 0" base_rpy="0 0 0" mesh_type="$(eval mesh_type)"/>
+<xacro:worm namespace="$(eval back_left)" parent_link="back_left_uib" base_xyz="0 0 0" base_rpy="0 0 0" mesh_type="$(eval mesh_type)"/>
+<xacro:worm namespace="$(eval back_right)" parent_link="back_right_uib" base_xyz="0 0 0" base_rpy="0 0 0" mesh_type="$(eval mesh_type)"/>
 <!-- Attach a foot module to each worm -->
-<xacro:rubber_foot namespace="$(eval front_left)" parent_link="$(eval front_left)_end_uib"/>
-<xacro:rubber_foot namespace="$(eval front_right)" parent_link="$(eval front_right)_end_uib"/>
-<xacro:rubber_foot namespace="$(eval back_left)" parent_link="$(eval back_left)_end_uib"/>
-<xacro:rubber_foot namespace="$(eval back_right)" parent_link="$(eval back_right)_end_uib"/>
+<xacro:rubber_foot namespace="$(eval front_left)" parent_link="$(eval front_left)_end_uib" mesh_type="$(eval mesh_type)"/>
+<xacro:rubber_foot namespace="$(eval front_right)" parent_link="$(eval front_right)_end_uib" mesh_type="$(eval mesh_type)"/>
+<xacro:rubber_foot namespace="$(eval back_left)" parent_link="$(eval back_left)_end_uib" mesh_type="$(eval mesh_type)"/>
+<xacro:rubber_foot namespace="$(eval back_right)" parent_link="$(eval back_right)_end_uib" mesh_type="$(eval mesh_type)"/>
 </robot>
