Commit message: Update damping coefficient to account for gear ratio

File: XACRO/3dof-worm.macro.xacro (robot description, xacro)
@@ -8,5 +8,5 @@
     <xacro:property name="motor_effort_limit" value="120"/>
     <xacro:property name="motor_velocity_limit" value="5.02654824"/>
-    <xacro:property name="motor_damping" value="0.8487"/>
+    <xacro:property name="motor_damping" value="0.0028"/>
     <xacro:property name="motor_gear_ratio" value="64"/>
     <xacro:property name="motor_rotor_inertia" value="0.00005645"/>

Commit message: Rollback motor damping change, model seems highly underdamped compared to real motors

File: XACRO/3dof-worm.macro.xacro (robot description, xacro)
@@ -15,5 +15,5 @@
     <xacro:property name="motor_effort_limit" value="120"/>
     <xacro:property name="motor_velocity_limit" value="5.02654824"/>
-    <xacro:property name="motor_damping" value="0.0028"/>
+    <xacro:property name="motor_damping" value="0.8487"/>
     <xacro:property name="motor_gear_ratio" value="64"/>
     <xacro:property name="motor_rotor_inertia" value="0.00005645"/>
