Commit message: Add hexapod xacro

File: XACRO/MACRO/3dof-worm.macro.xacro (robot description, xacro)
@@ -10,4 +10,5 @@
 <!-- |      base_xyz: translational offset of uib, ex: "0.2 0.1 0.1"                   | -->
 <!-- |      base_rpy: rotational offset of uib, "0.2 0.1 0.1"                          | -->
+<!-- |      mesh_type: type of mesh to link against, GLTF or OBJ                       | -->
 <!-- =================================================================================== -->
 <xacro:macro name="worm" params="namespace parent_link base_xyz base_rpy mesh_type">

File: XACRO/MACRO/pallets.macro.xacro (robot description, xacro)
@@ -12,4 +12,5 @@
 <!-- |    Args:                                                                        | -->
 <!-- |      spawn_z: height (in m) to spawn the pallet at                              | -->
+<!-- |      mesh_type: type of mesh to link against, GLTF or OBJ                       | -->
 <!-- =================================================================================== -->
 <xacro:macro name="turtle" params="spawn_z mesh_type">
@@ -92,3 +93,84 @@
     <link name="back_center_uib"/>
 </xacro:macro>
+<!-- =================================================================================== -->
+<!-- |    Macro for a hexapod pallet with six uib attachment points.                   | -->
+<!-- |    Downstream Links:                                                            | -->
+<!-- |      front_left_uib                                                             | -->
+<!-- |      front_right_uib                                                            | -->
+<!-- |      middle_left_uib                                                            | -->
+<!-- |      middle_right_uib                                                           | -->
+<!-- |      back_left_uib                                                              | -->
+<!-- |      back_right_uib                                                             | -->
+<!-- |    Args:                                                                        | -->
+<!-- |      spawn_z: height (in m) to spawn the pallet at                              | -->
+<!-- |      mesh_type: type of mesh to link against, GLTF or OBJ                       | -->
+<!-- =================================================================================== -->
+<xacro:macro name="hexapod" params="spawn_z mesh_type">
+    <!-- Virtual link to offset the body by some fixed amount -->
+    <link name="virtual_hexapod_body"/>
+    <joint name="virtual_hexapod_body_joint_fixed" type="fixed">
+        <parent link="virtual_hexapod_body"/>
+        <child link="hexapod_body"/>
+        <origin xyz="0 0 ${spawn_z}"/>
+    </joint>
+    <!-- Main pallet -->
+    <link name="hexapod_body">
+        <inertial>
+            <origin xyz="0 0 -0.13" rpy="0 0 -1.57"/>
+            <mass value="11.16"/>
+            <inertia ixx="1.65" ixy="0" ixz="0" iyy="0.78" iyz="0" izz="2.36"/>
+        </inertial>
+        <visual>
+            <origin xyz="0 0 0" rpy="0 0 -1.57"/>
+            <geometry>
+                <mesh filename="../Meshes/${mesh_type}/hexapod-pallet.gltf"/>
+            </geometry>
+        </visual>
+        <collision name="turtle_top_collision">
+            <origin xyz="0 0 0.062" rpy="0 0 0"/>
+            <geometry>
+                <box size="0.8 0.4 0.15"/>
+            </geometry>
+        </collision>
+    </link>
+    <!-- Front UIBs -->
+    <joint name="front_left_uib_joint_fixed" type="fixed">
+        <parent link="hexapod_body"/>
+        <child link="front_left_uib"/>
+        <origin xyz="0.328 0.204 0.062" rpy="-1.57 1.57 0"/>
+    </joint>
+    <link name="front_left_uib"/>
+    <joint name="front_right_uib_joint_fixed" type="fixed">
+        <parent link="hexapod_body"/>
+        <child link="front_right_uib"/>
+        <origin xyz="0.328 -0.204 0.062" rpy="1.57 -1.57 0"/>
+    </joint>
+    <link name="front_right_uib"/>
+    <!-- Middle UIBs -->
+    <joint name="middle_left_uib_joint_fixed" type="fixed">
+        <parent link="hexapod_body"/>
+        <child link="middle_left_uib"/>
+        <origin xyz="0.395 0 0.062" rpy="0 -1.57 3.14"/>
+    </joint>
+    <link name="middle_left_uib"/>
+    <joint name="middle_right_uib_joint_fixed" type="fixed">
+        <parent link="hexapod_body"/>
+        <child link="middle_right_uib"/>
+        <origin xyz="-0.395 0 0.062" rpy="0 -1.57 0"/>
+    </joint>
+    <link name="middle_right_uib"/>
+    <!-- Back UIBs -->
+    <joint name="back_left_uib_joint_fixed" type="fixed">
+        <parent link="hexapod_body"/>
+        <child link="back_left_uib"/>
+        <origin xyz="-0.328 0.204 0.062" rpy="-1.57 1.57 0"/>
+    </joint>
+    <link name="back_left_uib"/>
+    <joint name="back_right_uib_joint_fixed" type="fixed">
+        <parent link="hexapod_body"/>
+        <child link="back_right_uib"/>
+        <origin xyz="-0.328 -0.204 0.062" rpy="1.57 -1.57 0"/>
+    </joint>
+    <link name="back_right_uib"/>
+</xacro:macro>
 </robot>

File: XACRO/MACRO/species.macro.xacro (robot description, xacro)
@@ -6,4 +6,5 @@
 <!-- |      namespace: namespace to ensure uniqueness of names                         | -->
 <!-- |      parent_link: link name to affix the uib of this module to                  | -->
+<!-- |      mesh_type: type of mesh to link against, GLTF or OBJ                       | -->
 <!-- =================================================================================== -->
 <xacro:macro name="rubber_foot" params="namespace parent_link mesh_type">
