Commit message: Convert to ROS package for discovery

File: urdf/pony-worm.urdf (robot description, URDF)
Before this commit: robot worm, 6 links, 6 joints
Links:
- link pony_link_0: geometry collision cylinder length=0.075 radius=0.06; collision cylinder length=0.11 radius=0.075
- link pony_link_1: geometry collision box size=0.1 0.08 0.22; collision cylinder length=0.075 radius=0.06
- link pony_link_2: geometry collision box size=0.08 0.1 0.18; collision cylinder length=0.075 radius=0.06
- link pony_link_3: geometry collision box size=0.11 0.15 0.45; collision cylinder length=0.08 radius=0.075

File: urdf/turtle.urdf (robot description, URDF)
Before this commit: robot turtle, 36 links, 35 joints
Links:
- link duck_link_0: geometry collision cylinder length=0.075 radius=0.06; collision cylinder length=0.11 radius=0.075
- link duck_link_1: geometry collision box size=0.1 0.08 0.22; collision cylinder length=0.075 radius=0.06
- link duck_link_2: geometry collision box size=0.08 0.1 0.18; collision cylinder length=0.075 radius=0.06
- link duck_link_3: geometry collision box size=0.11 0.15 0.45; collision cylinder length=0.08 radius=0.075
- link duck_rubber_foot: geometry collision cylinder length=0.018 radius=0.115; collision cylinder length=0.05 radius=0.07
- link frog_link_0: geometry collision cylinder length=0.075 radius=0.06; collision cylinder length=0.11 radius=0.075
- link frog_link_1: geometry collision box size=0.1 0.08 0.22; collision cylinder length=0.075 radius=0.06
- link frog_link_2: geometry collision box size=0.08 0.1 0.18; collision cylinder length=0.075 radius=0.06
- link frog_link_3: geometry collision box size=0.11 0.15 0.45; collision cylinder length=0.08 radius=0.075
- link frog_rubber_foot: geometry collision cylinder length=0.018 radius=0.115; collision cylinder length=0.05 radius=0.07
- link lion_link_0: geometry collision cylinder length=0.075 radius=0.06; collision cylinder length=0.11 radius=0.075
- link lion_link_1: geometry collision box size=0.1 0.08 0.22; collision cylinder length=0.075 radius=0.06
- link lion_link_2: geometry collision box size=0.08 0.1 0.18; collision cylinder length=0.075 radius=0.06
- link lion_link_3: geometry collision box size=0.11 0.15 0.45; collision cylinder length=0.08 radius=0.075
- link lion_rubber_foot: geometry collision cylinder length=0.018 radius=0.115; collision cylinder length=0.05 radius=0.07
- link pony_link_0: geometry collision cylinder length=0.075 radius=0.06; collision cylinder length=0.11 radius=0.075
- link pony_link_1: geometry collision box size=0.1 0.08 0.22; collision cylinder length=0.075 radius=0.06
- link pony_link_2: geometry collision box size=0.08 0.1 0.18; collision cylinder length=0.075 radius=0.06
- link pony_link_3: geometry collision box size=0.11 0.15 0.45; collision cylinder length=0.08 radius=0.075
- link pony_rubber_foot: geometry collision cylinder length=0.018 radius=0.115; collision cylinder length=0.05 radius=0.07
- link turtle_body: geometry collision box size=0.11 0.11 0.4; collision box size=0.8 0.4 0.02

File: xacro/3dof-worm.urdf.xacro (robot description, xacro)
@@ -3,10 +3,10 @@
 <!-- Arguments -->
 <xacro:arg name="name" default=""/>
-<xacro:arg name="mesh_type" default="GLTF"/>
+<xacro:arg name="mesh_type" default="gltf"/>
 <xacro:if value="$(eval name == '')">
     <xacro:error msg="'name' was not provided"/>
 </xacro:if>
 <!-- Include xacro files -->
-<xacro:include filename="MACRO/3dof-worm.macro.xacro"/>
+<xacro:include filename="macros/3dof-worm.macro.xacro"/>
 <!-- Create a default worm fixed at the origin with the name passed -->
 <xacro:worm namespace="$(eval name)" parent_link="world" base_xyz="0 0 0" base_rpy="0 0 0" mesh_type="$(eval mesh_type)"/>

File: xacro/hexapod.urdf.xacro (robot description, xacro)
@@ -8,9 +8,9 @@
 <xacro:arg name="back_left" default="lion"/>
 <xacro:arg name="back_right" default="pony"/>
-<xacro:arg name="mesh_type" default="GLTF"/>
+<xacro:arg name="mesh_type" default="gltf"/>
 <!-- Include xacro files -->
-<xacro:include filename="MACRO/3dof-worm.macro.xacro"/>
-<xacro:include filename="MACRO/pallets.macro.xacro"/>
-<xacro:include filename="MACRO/species.macro.xacro"/>
+<xacro:include filename="macros/3dof-worm.macro.xacro"/>
+<xacro:include filename="macros/pallets.macro.xacro"/>
+<xacro:include filename="macros/species.macro.xacro"/>
 <!-- Create a hexapod pallet and attach worms to each corner uib -->
 <xacro:hexapod spawn_z="1.35" mesh_type="$(eval mesh_type)"/>

File: xacro/macros/3dof-worm.macro.xacro (robot description, xacro)
@@ -10,5 +10,5 @@
 <!-- |      base_xyz: translational offset of uib, ex: "0.2 0.1 0.1"                   | -->
 <!-- |      base_rpy: rotational offset of uib, "0.2 0.1 0.1"                          | -->
-<!-- |      mesh_type: type of mesh to link against, GLTF or OBJ                       | -->
+<!-- |      mesh_type: type of mesh to link against, gltf or obj                       | -->
 <!-- =================================================================================== -->
 <xacro:macro name="worm" params="namespace parent_link base_xyz base_rpy mesh_type">
@@ -40,5 +40,5 @@
             <origin xyz="0 0 0.045" rpy="0 0 0"/>
             <geometry>
-                <mesh filename="../Meshes/${mesh_type}/link-0.gltf"/>
+                <mesh filename="../meshes/${mesh_type}/link-0.gltf"/>
             </geometry>
         </visual>
@@ -73,5 +73,5 @@
             <origin xyz="0.05 0 0" rpy="0 0 -1.57"/>
             <geometry>
-                <mesh filename="../Meshes/${mesh_type}/link-1.gltf"/>
+                <mesh filename="../meshes/${mesh_type}/link-1.gltf"/>
             </geometry>
         </visual>
@@ -106,5 +106,5 @@
             <origin xyz="0 -0.05 0" rpy="0 0 3.14"/>
             <geometry>
-                <mesh filename="../Meshes/${mesh_type}/link-2.gltf"/>
+                <mesh filename="../meshes/${mesh_type}/link-2.gltf"/>
             </geometry>
         </visual>
@@ -139,5 +139,5 @@
             <origin xyz="0 -0.05 0" rpy="0 0 1.57"/>
             <geometry>
-                <mesh filename="../Meshes/${mesh_type}/link-3.gltf"/>
+                <mesh filename="../meshes/${mesh_type}/link-3.gltf"/>
             </geometry>
         </visual>

File: xacro/macros/pallets.macro.xacro (robot description, xacro)
@@ -12,5 +12,5 @@
 <!-- |    Args:                                                                        | -->
 <!-- |      spawn_z: height (in m) to spawn the pallet at                              | -->
-<!-- |      mesh_type: type of mesh to link against, GLTF or OBJ                       | -->
+<!-- |      mesh_type: type of mesh to link against, gltf or obj                       | -->
 <!-- =================================================================================== -->
 <xacro:macro name="turtle" params="spawn_z mesh_type">
@@ -32,5 +32,5 @@
             <origin xyz="0 0 0" rpy="0 0 -1.57"/>
             <geometry>
-                <mesh filename="../Meshes/${mesh_type}/turtle-pallet.gltf"/>
+                <mesh filename="../meshes/${mesh_type}/turtle-pallet.gltf"/>
             </geometry>
         </visual>
@@ -104,5 +104,5 @@
 <!-- |    Args:                                                                        | -->
 <!-- |      spawn_z: height (in m) to spawn the pallet at                              | -->
-<!-- |      mesh_type: type of mesh to link against, GLTF or OBJ                       | -->
+<!-- |      mesh_type: type of mesh to link against, gltf or obj                       | -->
 <!-- =================================================================================== -->
 <xacro:macro name="hexapod" params="spawn_z mesh_type">
@@ -124,5 +124,5 @@
             <origin xyz="0 0 0" rpy="0 0 -1.57"/>
             <geometry>
-                <mesh filename="../Meshes/${mesh_type}/hexapod-pallet.gltf"/>
+                <mesh filename="../meshes/${mesh_type}/hexapod-pallet.gltf"/>
             </geometry>
         </visual>

File: xacro/macros/species.macro.xacro (robot description, xacro)
@@ -6,5 +6,5 @@
 <!-- |      namespace: namespace to ensure uniqueness of names                         | -->
 <!-- |      parent_link: link name to affix the uib of this module to                  | -->
-<!-- |      mesh_type: type of mesh to link against, GLTF or OBJ                       | -->
+<!-- |      mesh_type: type of mesh to link against, gltf or obj                       | -->
 <!-- =================================================================================== -->
 <xacro:macro name="rubber_foot" params="namespace parent_link mesh_type">
@@ -21,5 +21,5 @@
         <visual>
             <geometry>
-                <mesh filename="../Meshes/${mesh_type}/rubber-foot.gltf"/>
+                <mesh filename="../meshes/${mesh_type}/rubber-foot.gltf"/>
             </geometry>
         </visual>

File: xacro/turtle.urdf.xacro (robot description, xacro)
@@ -6,9 +6,9 @@
 <xacro:arg name="back_left" default="lion"/>
 <xacro:arg name="back_right" default="pony"/>
-<xacro:arg name="mesh_type" default="GLTF"/>
+<xacro:arg name="mesh_type" default="gltf"/>
 <!-- Include xacro files -->
-<xacro:include filename="MACRO/3dof-worm.macro.xacro"/>
-<xacro:include filename="MACRO/pallets.macro.xacro"/>
-<xacro:include filename="MACRO/species.macro.xacro"/>
+<xacro:include filename="macros/3dof-worm.macro.xacro"/>
+<xacro:include filename="macros/pallets.macro.xacro"/>
+<xacro:include filename="macros/species.macro.xacro"/>
 <!-- Create a turtle pallet and attach worms to each corner uib -->
 <xacro:turtle spawn_z="1.35" mesh_type="$(eval mesh_type)"/>
