Commit message: Add working hexapod body

File: urdf/hexapod.urdf (robot description, URDF)
Before this commit: robot turtle, 36 links, 35 joints
Links:
- removed link back_center_uib
- removed link front_center_uib
- removed link turtle_body
- removed link virtual_turtle_body
- added link hare_base
- added link hare_end_uib
- added link hare_link_0, mass 1.59; collision cylinder length=0.075 radius=0.06; collision cylinder length=0.11 radius=0.075
- added link hare_link_1, mass 1.59; collision box size=0.1 0.08 0.22; collision cylinder length=0.075 radius=0.06
- added link hare_link_2, mass 1.59; collision box size=0.08 0.1 0.18; collision cylinder length=0.075 radius=0.06
- added link hare_link_3, mass 5.00; collision box size=0.11 0.15 0.45; collision cylinder length=0.08 radius=0.075
- added link hare_rubber_foot, mass 1.54; collision cylinder length=0.018 radius=0.115; collision cylinder length=0.05 radius=0.07
- added link hexapod_body, mass 11.144; collision box size=0.5 0.7 0.15; collision box size=0.5 0.7 0.15
- added link middle_left_uib
- added link middle_right_uib
- added link seal_base
- added link seal_end_uib
- added link seal_link_0, mass 1.59; collision cylinder length=0.075 radius=0.06; collision cylinder length=0.11 radius=0.075
- added link seal_link_1, mass 1.59; collision box size=0.1 0.08 0.22; collision cylinder length=0.075 radius=0.06
- added link seal_link_2, mass 1.59; collision box size=0.08 0.1 0.18; collision cylinder length=0.075 radius=0.06
- added link seal_link_3, mass 5.00; collision box size=0.11 0.15 0.45; collision cylinder length=0.08 radius=0.075
- added link seal_rubber_foot, mass 1.54; collision cylinder length=0.018 radius=0.115; collision cylinder length=0.05 radius=0.07
- added link virtual_hexapod_body
Joints:
- removed joint back_center_uib_joint_fixed
- removed joint front_center_uib_joint_fixed
- removed joint virtual_turtle_body_joint_fixed
- added joint hare_base_joint_fixed: type fixed, parent hare_base, child hare_link_0
- added joint hare_end_uib_joint_fixed: type fixed, parent hare_link_3, child hare_end_uib, origin xyz=0 -0.012 0.498 rpy=3.14 0 -0.35
- added joint hare_joint_0: type revolute, parent hare_link_0, child hare_link_1, origin xyz=0 0 0.145 rpy=0 0 0, axis 1 0 0, limit lower=-2.094 upper=2.094 effort=120 velocity=5.02654824
- added joint hare_joint_1: type revolute, parent hare_link_1, child hare_link_2, origin xyz=0 0 0.25 rpy=0 0 0, axis 0 1 0, limit lower=-2.094 upper=2.094 effort=120 velocity=5.02654824
- added joint hare_joint_2: type revolute, parent hare_link_2, child hare_link_3, origin xyz=0 0 0.22 rpy=0 0 0, axis 0 1 0, limit lower=-2.094 upper=2.094 effort=120 velocity=5.02654824
- added joint hare_rubber_foot_joint_fixed: type fixed, parent hare_end_uib, child hare_rubber_foot
- added joint hare_uib_joint_fixed: type fixed, parent middle_right_uib, child hare_base, origin xyz=0 0 0 rpy=0 0 0
- added joint middle_left_uib_joint_fixed: type fixed, parent hexapod_body, child middle_left_uib, origin xyz=0 0.5 -0.064 rpy=-1.57 1.57 0
- added joint middle_right_uib_joint_fixed: type fixed, parent hexapod_body, child middle_right_uib, origin xyz=0 -0.5 -0.064 rpy=1.57 -1.57 0
- added joint seal_base_joint_fixed: type fixed, parent seal_base, child seal_link_0
- added joint seal_end_uib_joint_fixed: type fixed, parent seal_link_3, child seal_end_uib, origin xyz=0 -0.012 0.498 rpy=3.14 0 -0.35
- added joint seal_joint_0: type revolute, parent seal_link_0, child seal_link_1, origin xyz=0 0 0.145 rpy=0 0 0, axis 1 0 0, limit lower=-2.094 upper=2.094 effort=120 velocity=5.02654824
- added joint seal_joint_1: type revolute, parent seal_link_1, child seal_link_2, origin xyz=0 0 0.25 rpy=0 0 0, axis 0 1 0, limit lower=-2.094 upper=2.094 effort=120 velocity=5.02654824
- added joint seal_joint_2: type revolute, parent seal_link_2, child seal_link_3, origin xyz=0 0 0.22 rpy=0 0 0, axis 0 1 0, limit lower=-2.094 upper=2.094 effort=120 velocity=5.02654824
- added joint seal_rubber_foot_joint_fixed: type fixed, parent seal_end_uib, child seal_rubber_foot
- added joint seal_uib_joint_fixed: type fixed, parent middle_left_uib, child seal_base, origin xyz=0 0 0 rpy=0 0 0
- added joint virtual_hexapod_body_joint_fixed: type fixed, parent virtual_hexapod_body, child hexapod_body, origin xyz=0 0 1.35
- joint back_left_uib_joint_fixed: origin xyz=-0.328 0.204 0.062 rpy=-1.57 1.57 0 -> xyz=-0.6 0.086 -0.064 rpy=-1.57 1.57 0; parent turtle_body -> hexapod_body
- joint back_right_uib_joint_fixed: origin xyz=-0.328 -0.204 0.062 rpy=1.57 -1.57 0 -> xyz=-0.6 -0.086 -0.064 rpy=1.57 -1.57 0; parent turtle_body -> hexapod_body
- joint front_left_uib_joint_fixed: origin xyz=0.328 0.204 0.062 rpy=-1.57 1.57 0 -> xyz=0.6 0.086 -0.064 rpy=-1.57 1.57 0; parent turtle_body -> hexapod_body
- joint front_right_uib_joint_fixed: origin xyz=0.328 -0.204 0.062 rpy=1.57 -1.57 0 -> xyz=0.6 -0.086 -0.064 rpy=1.57 -1.57 0; parent turtle_body -> hexapod_body

File: xacro/macros/pallets.macro.xacro (robot description, xacro)
@@ -27,5 +27,5 @@
             <origin xyz="0 0 -0.13" rpy="0 0 -1.57"/>
             <mass value="21.89"/>
-            <inertia ixx="0.9" ixy="0" ixz="0" iyy="1.5" iyz="0" izz="1.0"/>
+            <inertia ixx="1.5" ixy="0" ixz="0" iyy="0.9" iyz="0" izz="1.0"/>
         </inertial>
         <visual>
@@ -117,7 +117,7 @@
     <link name="hexapod_body">
         <inertial>
-            <origin xyz="0 0 -0.13" rpy="0 0 -1.57"/>
-            <mass value="11.16"/>
-            <inertia ixx="1.65" ixy="0" ixz="0" iyy="0.78" iyz="0" izz="2.36"/>
+        <origin rpy="0 0 -1.57" xyz="0 0 -0.064"/>
+        <mass value="11.144"/>
+        <inertia ixx="1.654" ixy="0" ixz="0" iyy="0.779" iyz="0" izz="2.362"/>
         </inertial>
         <visual>
@@ -127,8 +127,26 @@
             </geometry>
         </visual>
-        <collision name="turtle_top_collision">
-            <origin xyz="0 0 0.062" rpy="0 0 0"/>
+        <collision name="hexapod_front_left_collision">
+            <origin rpy="0 0 0.959931" xyz="0.2 0.1 -0.064"/>
             <geometry>
-                <box size="0.8 0.4 0.15"/>
+                <box size="0.5 0.7 0.15"/>
+            </geometry>
+        </collision>
+        <collision name="hexapod_front_right_collision">
+            <origin rpy="0 0 -0.959931" xyz="0.2 -0.1 -0.064"/>
+            <geometry>
+                <box size="0.5 0.7 0.15"/>
+            </geometry>
+        </collision>
+        <collision name="hexapod_back_left_collision">
+            <origin rpy="0 0 -0.959931" xyz="-0.2 0.1 -0.064"/>
+            <geometry>
+                <box size="0.5 0.7 0.15"/>
+            </geometry>
+        </collision>
+        <collision name="hexapod_back_right_collision">
+            <origin rpy="0 0 0.959931" xyz="-0.2 -0.1 -0.064"/>
+            <geometry>
+                <box size="0.5 0.7 0.15"/>
             </geometry>
         </collision>
@@ -138,5 +156,5 @@
         <parent link="hexapod_body"/>
         <child link="front_left_uib"/>
-        <origin xyz="0.328 0.204 0.062" rpy="-1.57 1.57 0"/>
+        <origin xyz="0.6 0.086 -0.064" rpy="-1.57 1.57 0"/>
     </joint>
     <link name="front_left_uib"/>
@@ -144,5 +162,5 @@
         <parent link="hexapod_body"/>
         <child link="front_right_uib"/>
-        <origin xyz="0.328 -0.204 0.062" rpy="1.57 -1.57 0"/>
+        <origin xyz="0.6 -0.086 -0.064" rpy="1.57 -1.57 0"/>
     </joint>
     <link name="front_right_uib"/>
@@ -151,5 +169,5 @@
         <parent link="hexapod_body"/>
         <child link="middle_left_uib"/>
-        <origin xyz="0.395 0 0.062" rpy="0 -1.57 3.14"/>
+        <origin xyz="0 0.5 -0.064" rpy="-1.57 1.57 0"/>
     </joint>
     <link name="middle_left_uib"/>
@@ -157,5 +175,5 @@
         <parent link="hexapod_body"/>
         <child link="middle_right_uib"/>
-        <origin xyz="-0.395 0 0.062" rpy="0 -1.57 0"/>
+        <origin xyz="0 -0.5 -0.064" rpy="1.57 -1.57 0"/>
     </joint>
     <link name="middle_right_uib"/>
@@ -164,5 +182,5 @@
         <parent link="hexapod_body"/>
         <child link="back_left_uib"/>
-        <origin xyz="-0.328 0.204 0.062" rpy="-1.57 1.57 0"/>
+        <origin xyz="-0.6 0.086 -0.064" rpy="-1.57 1.57 0"/>
     </joint>
     <link name="back_left_uib"/>
@@ -170,5 +188,5 @@
         <parent link="hexapod_body"/>
         <child link="back_right_uib"/>
-        <origin xyz="-0.328 -0.204 0.062" rpy="1.57 -1.57 0"/>
+        <origin xyz="-0.6 -0.086 -0.064" rpy="1.57 -1.57 0"/>
     </joint>
     <link name="back_right_uib"/>
