Commit message: Make macro fields optional

File: xacro/macros/3dof-worm.macro.xacro (robot description, xacro)
@@ -8,9 +8,9 @@
 <!-- |      namespace: namespace that this worm publishes to                           | -->
 <!-- |      parent_link: link name to affix the uib of this worm to                    | -->
-<!-- |      base_xyz: translational offset of uib, ex: "0.2 0.1 0.1"                   | -->
-<!-- |      base_rpy: rotational offset of uib, "0.2 0.1 0.1"                          | -->
-<!-- |      mesh_type: type of mesh to link against, gltf or obj                       | -->
+<!-- |      base_xyz (optional): translational offset of uib, ex: "0.2 0.1 0.1"        | -->
+<!-- |      base_rpy (optional): rotational offset of uib, "0.2 0.1 0.1"               | -->
+<!-- |      mesh_type (optional): type of mesh to link against, gltf or obj            | -->
 <!-- =================================================================================== -->
-<xacro:macro name="worm" params="namespace parent_link base_xyz base_rpy mesh_type">
+<xacro:macro name="worm" params="namespace parent_link base_xyz:=0_0_0 base_rpy:=0_0_0 mesh_type:=obj">
     <!-- Local parameters -->
     <xacro:property name="motor_collision_length" value="0.075"/>

File: xacro/macros/pallets.macro.xacro (robot description, xacro)
@@ -11,8 +11,8 @@
 <!-- |      back_center_uib                                                            | -->
 <!-- |    Args:                                                                        | -->
-<!-- |      spawn_z: height (in m) to spawn the pallet at                              | -->
-<!-- |      mesh_type: type of mesh to link against, gltf or obj                       | -->
+<!-- |      spawn_z (optional): height (in m) to spawn the pallet at                   | -->
+<!-- |      mesh_type (optional): type of mesh to link against, gltf or obj            | -->
 <!-- =================================================================================== -->
-<xacro:macro name="turtle" params="spawn_z mesh_type">
+<xacro:macro name="turtle" params="spawn_z:=0 mesh_type:=obj">
     <!-- Virtual link to offset the body by some fixed amount -->
     <link name="virtual_turtle_body"/>
@@ -103,8 +103,8 @@
 <!-- |      back_right_uib                                                             | -->
 <!-- |    Args:                                                                        | -->
-<!-- |      spawn_z: height (in m) to spawn the pallet at                              | -->
-<!-- |      mesh_type: type of mesh to link against, gltf or obj                       | -->
+<!-- |      spawn_z (optional): height (in m) to spawn the pallet at                   | -->
+<!-- |      mesh_type (optional): type of mesh to link against, gltf or obj            | -->
 <!-- =================================================================================== -->
-<xacro:macro name="hexapod" params="spawn_z mesh_type">
+<xacro:macro name="hexapod" params="spawn_z:=0 mesh_type:=obj">
     <!-- Virtual link to offset the body by some fixed amount -->
     <link name="virtual_hexapod_body"/>

File: xacro/macros/species.macro.xacro (robot description, xacro)
@@ -6,7 +6,7 @@
 <!-- |      namespace: namespace to ensure uniqueness of names                         | -->
 <!-- |      parent_link: link name to affix the uib of this module to                  | -->
-<!-- |      mesh_type: type of mesh to link against, gltf or obj                       | -->
+<!-- |      mesh_type (optional): type of mesh to link against, gltf or obj            | -->
 <!-- =================================================================================== -->
-<xacro:macro name="rubber_foot" params="namespace parent_link mesh_type">
+<xacro:macro name="rubber_foot" params="namespace parent_link mesh_type:=obj">
     <joint name="${namespace}_rubber_foot_joint_fixed" type="fixed">
         <parent link="${parent_link}"/>
